Commit message: Adding transmission.

File: robots/robotiq_arg85.transmission.xacro (robot description, xacro)
@@ -4,5 +4,5 @@
     <transmission name="finger_joint_trans">
       <type>transmission_interface/SimpleTransmission</type>
-      <joint name=" finger_joint">
+      <joint name="finger_joint">
         <hardwareInterface>PositionJointInterface</hardwareInterface>
       </joint>

File: robots/robotiq_arg85_description.urdf.xacro (robot description, xacro)
@@ -308,3 +308,4 @@
     <axis xyz="0 1 0" />
   </joint>
+    <xacro:robotiq_arg85_transmission/>
 </robot>
